Commit message: Fix detection node: remove cv_bridge dependency, wrap EigenTrajectory import

File: ros2_ws/src/g1_description/urdf/g1_29dof.urdf (robot description, URDF)
Before this commit: robot g1_29dof, 40 links, 39 joints
Links:
- link head_link: geometry collision mesh filename=package://g1_description/urdf/meshes/head_link.STL; visual mesh filename=package://g1_description/urdf/meshes/head_link.STL
- link left_ankle_pitch_link: geometry collision mesh filename=package://g1_description/urdf/meshes/left_ankle_pitch_link.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; visual mesh filename=package://g1_description/urdf/meshes/left_ankle_pitch_link.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
- link left_ankle_roll_link: geometry collision sphere radius=0.005; collision sphere radius=0.005
- link left_elbow_link: geometry collision mesh filename=package://g1_description/urdf/meshes/left_elbow_link.STL; visual mesh filename=package://g1_description/urdf/meshes/left_elbow_link.STL
- link left_hip_pitch_link: geometry collision mesh filename=package://g1_description/urdf/meshes/left_hip_pitch_link.STL; visual mesh filename=package://g1_description/urdf/meshes/left_hip_pitch_link.STL
- link left_hip_roll_link: geometry collision mesh filename=package://g1_description/urdf/meshes/left_hip_roll_link.STL; visual mesh filename=package://g1_description/urdf/meshes/left_hip_roll_link.STL
- link left_hip_yaw_link: geometry collision mesh filename=package://g1_description/urdf/meshes/left_hip_yaw_link.STL; visual mesh filename=package://g1_description/urdf/meshes/left_hip_yaw_link.STL
- link left_knee_link: geometry collision mesh filename=package://g1_description/urdf/meshes/left_knee_link.STL; visual mesh filename=package://g1_description/urdf/meshes/left_knee_link.STL
- link left_rubber_hand: geometry visual mesh filename=package://g1_description/urdf/meshes/left_rubber_hand.STL
- link left_shoulder_pitch_link: geometry collision cylinder length=0.05 radius=0.03; visual mesh filename=package://g1_description/urdf/meshes/left_shoulder_pitch_li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
- link left_shoulder_roll_link: geometry collision cylinder length=0.03 radius=0.03; visual mesh filename=package://g1_description/urdf/meshes/left_shoulder_roll_lin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
- link left_shoulder_yaw_link: geometry collision mesh filename=package://g1_description/urdf/meshes/left_shoulder_yaw_link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; visual mesh filename=package://g1_description/urdf/meshes/left_shoulder_yaw_link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
- link left_wrist_pitch_link: geometry collision mesh filename=package://g1_description/urdf/meshes/left_wrist_pitch_link.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; visual mesh filename=package://g1_description/urdf/meshes/left_wrist_pitch_link.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
- link left_wrist_roll_link: geometry collision mesh filename=package://g1_description/urdf/meshes/left_wrist_roll_link.S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; visual mesh filename=package://g1_description/urdf/meshes/left_wrist_roll_link.S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
- link left_wrist_yaw_link: geometry collision mesh filename=package://g1_description/urdf/meshes/left_wrist_yaw_link.STL; visual mesh filename=package://g1_description/urdf/meshes/left_wrist_yaw_link.STL
- link logo_link: geometry collision mesh filename=package://g1_description/urdf/meshes/logo_link.STL; visual mesh filename=package://g1_description/urdf/meshes/logo_link.STL
- link pelvis: geometry visual mesh filename=package://g1_description/urdf/meshes/pelvis.STL
- link pelvis_contour_link: geometry collision mesh filename=package://g1_description/urdf/meshes/pelvis_contour_link.STL; visual mesh filename=package://g1_description/urdf/meshes/pelvis_contour_link.STL
- link right_ankle_pitch_link: geometry collision mesh filename=package://g1_description/urdf/meshes/right_ankle_pitch_link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; visual mesh filename=package://g1_description/urdf/meshes/right_ankle_pitch_link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
- link right_ankle_roll_link: geometry collision sphere radius=0.005; collision sphere radius=0.005
- link right_elbow_link: geometry collision mesh filename=package://g1_description/urdf/meshes/right_elbow_link.STL; visual mesh filename=package://g1_description/urdf/meshes/right_elbow_link.STL
- link right_hip_pitch_link: geometry collision mesh filename=package://g1_description/urdf/meshes/right_hip_pitch_link.S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; visual mesh filename=package://g1_description/urdf/meshes/right_hip_pitch_link.S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
- link right_hip_roll_link: geometry collision mesh filename=package://g1_description/urdf/meshes/right_hip_roll_link.STL; visual mesh filename=package://g1_description/urdf/meshes/right_hip_roll_link.STL
- link right_hip_yaw_link: geometry collision mesh filename=package://g1_description/urdf/meshes/right_hip_yaw_link.STL; visual mesh filename=package://g1_description/urdf/meshes/right_hip_yaw_link.STL
- link right_knee_link: geometry collision mesh filename=package://g1_description/urdf/meshes/right_knee_link.STL; visual mesh filename=package://g1_description/urdf/meshes/right_knee_link.STL
- link right_rubber_hand: geometry visual mesh filename=package://g1_description/urdf/meshes/right_rubber_hand.STL
- link right_shoulder_pitch_link: geometry collision cylinder length=0.05 radius=0.03; visual mesh filename=package://g1_description/urdf/meshes/right_shoulder_pitch_l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
- link right_shoulder_roll_link: geometry collision cylinder length=0.03 radius=0.03; visual mesh filename=package://g1_description/urdf/meshes/right_shoulder_roll_li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
- link right_shoulder_yaw_link: geometry collision mesh filename=package://g1_description/urdf/meshes/right_shoulder_yaw_lin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; visual mesh filename=package://g1_description/urdf/meshes/right_shoulder_yaw_lin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
- link right_wrist_pitch_link: geometry collision mesh filename=package://g1_description/urdf/meshes/right_wrist_pitch_link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; visual mesh filename=package://g1_description/urdf/meshes/right_wrist_pitch_link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
- link right_wrist_roll_link: geometry collision mesh filename=package://g1_description/urdf/meshes/right_wrist_roll_link.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; visual mesh filename=package://g1_description/urdf/meshes/right_wrist_roll_link.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
- link right_wrist_yaw_link: geometry collision mesh filename=package://g1_description/urdf/meshes/right_wrist_yaw_link.S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; visual mesh filename=package://g1_description/urdf/meshes/right_wrist_yaw_link.S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
- link torso_link: geometry collision mesh filename=package://g1_description/urdf/meshes/torso_link.STL; visual mesh filename=package://g1_description/urdf/meshes/torso_link.STL
- link waist_roll_link: geometry visual mesh filename=package://g1_description/urdf/meshes/waist_roll_link.STL
- link waist_support_link: geometry collision mesh filename=package://g1_description/urdf/meshes/waist_support_link.STL; visual mesh filename=package://g1_description/urdf/meshes/waist_support_link.STL
- link waist_yaw_link: geometry visual mesh filename=package://g1_description/urdf/meshes/waist_yaw_link.STL
